File: projects/HSLink-Pro/hardware/HSLinkPro.kicad_sch (KiCad schematic)
At the start: 19 parts, among them J3 Header 1.27 4P, SW1 1TS028A-1900-0600-CT, U1 HPM5301IEG1, Y1 24M

Commit message: update: 更新原理图
Parts:
- added D2: 1N5819, Diode_SMD:D_SOD-523, symbol Device:D
- added R2: 100k, Resistor_SMD:R_0402_1005Metric, symbol Device:R
Connections:
- net +3V3: no longer C57.1, D1.1 (VDD)
- net GND: now also R2.2
- net PORT_EN: now reaches U1.1 (PA04/URT1.CTS/SPI0.CS0/TRGM0.P04/JTAG.TDO)
- net PORT_EN: now also R2.1
- new net: C57.1, D1.1 (VDD), D2.1 (K)
- new net +5V: D2.2 (A)
- no-connect marks 6 -> 5
Other:
- sheet Interface  ports: added none; removed POWER_OUT_EN
- sheet Power ports: added PORT_EN, P_EN; removed none
- moved on the sheet: SW1

Commit message: update: 1.2.0硬件
Connections:
- net BOOT0: no longer D1.4 (DIN)
- net UART_RTS: now also U1.48 (PA05/TMR1.COMP2/URT1.DE/URT1.RTS/SPI0.SCLK/TRGM0.P05/JTAG.TDI); no longer U1.46 (PA07/TMR0.COMP0/URT1.TXD/I2C1.SCL/SPI0.MOSI/TRGM0.P07/JTAG.TMS)
- new net WS2812: D1.4 (DIN), U1.46 (PA07/TMR0.COMP0/URT1.TXD/I2C1.SCL/SPI0.MOSI/TRGM0.P07/JTAG.TMS)
- no-connect marks 5 -> 4
Changed lines of the file:
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@@
 		(at 34.29 115.57)
 	)
-	(no_connect
-		(at 34.29 36.83)
-	)
 	(wire
 		(pts
@@
 	(wire
 		(pts
+			(xy 22.86 36.83) (xy 34.29 36.83)
+		)
+		(stroke
+			(width 0)
+			(type default)
+		)
+	)
+	(wire
+		(pts
 			(xy 22.86 144.78) (xy 30.48 144.78)
 		)
@@
 	(wire
 		(pts
-			(xy 60.96 171.45) (xy 67.31 171.45)
+			(xy 59.69 171.45) (xy 67.31 171.45)
 		)
 		(stroke
@@
 		)
 	)
-	(label "BOOT0"
-		(at 60.96 171.45 0)
-		(effects
-			(font
-				(size 1.27 1.27)
-			)
-			(justify left bottom)
-		)
-	)
-	(label "UART_RTS"
-		(at 22.86 41.91 0)
-		(effects
-			(font
-				(size 1.27 1.27)
-			)
-			(justify left bottom)
-		)
-	)
 	(label "ISP_TX"
 		(at 38.1 161.29 0)
@@
 		)
 	)
+	(label "WS2812"
+		(at 22.86 41.91 0)
+		(effects
+			(font
+				(size 1.27 1.27)
+			)
+			(justify left bottom)
+		)
+	)
 	(label "SWCLK{slash}TCK"
 		(at 22.86 59.69 0)
@@
 		)
 	)
+	(label "UART_RTS"
+		(at 22.86 36.83 0)
+		(effects
+			(font
+				(size 1.27 1.27)
+			)
+			(justify left bottom)
+		)
+	)
 	(label "PORT_EN"
 		(at 64.77 134.62 0)
@@
 		(effects
 			(font
+				(size 1.27 1.27)
+			)
+			(justify left bottom)
+		)
+	)
+	(label "WS2812"
+		(at 59.69 171.45 0)
+		(effects
+			(font
