File: projects/HSLink-Pro/hardware/HSLinkPro.kicad_sch (KiCad schematic)
At the start: 19 parts, among them J3 Header 1.27 4P, SW1 1TS028A-1900-0600-CT, U1 HPM5301IEG1, Y1 24M

Commit message: HSLink-Pro: 2.3.1 (#29)
* update: 更新电源部分

* update: 更新原理图

* update: 更新PCB

- 修改定位孔位置
- 修改Type-C位置

* update: 添加RTT LOGO

* chore: 添加cJSON库

* feat: 添加与上位机的HID通信接口

* refactor: 重构命令解析部分代码

* fix: 修复描述符错误

* feat: 添加上位机下发设置功能

* feat: 添加数据保存

* fix: 修复可能的一些错误

* fix: 修复写入flash死机问题

* fix: 潜在的内存泄露问题

* chore: 添加tlsf

* chore: 切换cJSON库位置

* feat: 内存管理切换为tlsf

* feat: 添加首次默认设置

* feat: 添加硬件版本号

* feat: 添加获取设置

* chore: 将项目修改为cpp

* feat: 重构为cpp

* fix: 修复release下可能会崩溃的玄学问题

* chore: 删除cJSON库

* fix: 修复RapidJSON库所需内存

* fix: 修复nickname设置问题

* fix: BL工程编译失败

* fix: BL工程里面关闭所有输出

* fix: 修复一些warning

* update: README

* fix: get_setting字段错误

* update: 1.2.0硬件

* style: 统一接口命名

* feat: 添加upgrade命令

* fix: 将硬件版本号放在OTP寄存器中

* fix: 解决初始值问题

* fix: PWM输出极性反了

* fix: 1.2.0硬件修改IO

* release: 2.3.1
Parts:
- added D2: 1N5819, Diode_SMD:D_SOD-523, symbol Device:D
- added R2: 100k, Resistor_SMD:R_0402_1005Metric, symbol Device:R
Connections:
- net +3V3: no longer C57.1, D1.1 (VDD)
- net BOOT0: no longer D1.4 (DIN)
- net GND: now also R2.2
- net UART_RTS: now also U1.48 (PA05/TMR1.COMP2/URT1.DE/URT1.RTS/SPI0.SCLK/TRGM0.P05/JTAG.TDI); no longer U1.46 (PA07/TMR0.COMP0/URT1.TXD/I2C1.SCL/SPI0.MOSI/TRGM0.P07/JTAG.TMS)
- net PORT_EN: now reaches U1.1 (PA04/URT1.CTS/SPI0.CS0/TRGM0.P04/JTAG.TDO)
- net PORT_EN: now also R2.1
- new net: C57.1, D1.1 (VDD), D2.1 (K)
- new net +5V: D2.2 (A)
- new net WS2812: D1.4 (DIN), U1.46 (PA07/TMR0.COMP0/URT1.TXD/I2C1.SCL/SPI0.MOSI/TRGM0.P07/JTAG.TMS)
- no-connect marks 6 -> 4
Other:
- sheet Interface  ports: added none; removed POWER_OUT_EN
- sheet Power ports: added PORT_EN, P_EN; removed none
- moved on the sheet: SW1
