File: projects/HSLink-Pro/hardware/Power.kicad_sch (KiCad schematic)
At the start: 44 parts, among them U1 HPM5301IEG1, U10 EA3036C, U13 LMV321

Commit message: update: 更新电源部分
Parts:
- removed C48: 10u, Capacitor_SMD:C_0402_1005Metric, symbol Device:C
- removed C49: 220p, Capacitor_SMD:C_0402_1005Metric, symbol Device:C
- removed C51: 10u, Capacitor_SMD:C_0603_1608Metric, symbol Device:C
- removed L3: 1.5u, Inductor_SMD:L_1008_2520Metric, symbol Device:L
- removed R2: 22.1k, Resistor_SMD:R_0402_1005Metric, symbol Device:R
- removed R3: 100k, Resistor_SMD:R_0402_1005Metric, symbol Device:R
- removed U10: EA3036C, Package_DFN_QFN:QFN-20-1EP_3x3mm_P0.4mm_EP1.65x1.65mm, symbol Regulator_Switching:EA3036C
- added U10: TLV62568DRL, Package_TO_SOT_SMD:SOT-563, symbol Regulator_Switching:TLV62568DRL
- C40: value 1u -> 4.7u
- C41, C46: value 10u -> 22u
- C47: value 10u -> 0.1u; footprint Capacitor_SMD:C_0603_1608Metric -> Capacitor_SMD:C_0402_1005Metric
- C50: value 220p -> 6.8p
- L1: footprint Inductor_SMD:L_1008_2520Metric -> Inductor_SMD:L_Murata_DFE201610P
- L2: value 1.5u -> 2.2uH; footprint Inductor_SMD:L_1008_2520Metric -> Inductor_SMD:L_Murata_DFE201610P
Connections:
- net +3V3: no longer L2.1
- net +5V: now also U10.3 (VIN), U10.5 (EN); no longer C41.1, C46.1, C47.1
- net GND: now also U10.2 (GND)
- net TRANS_VCC: now also C41.1, C46.1, C47.1, L2.2
- net TRANS_VREF: now also U10.1 (FB)
- new net: L2.1, U10.4 (SW)
- no-connect marks 3 -> 0

Commit message: update: 更新原理图
Parts:
- added C34: 0.1u, Capacitor_SMD:C_0402_1005Metric, symbol Device:C
- added C48, C49, C51, C59, C60, C61, C62, C63: 1u, Capacitor_SMD:C_0402_1005Metric, symbol Device:C
- added U19: ME6211C33U4G, Package_DFN_QFN:OnSemi_XDFN4-1EP_1.0x1.0mm_EP0.52x0.52mm, symbol Regulator_Linear:NCP115AMX120TCG
- added U20, U21, U22: AW3512, Package_CSP:WLCSP-4-X1-WLB0909-4_0.89x0.89mm_P0.5mm, symbol Power_Management:AP22913CN4
Connections:
- net +3V3: now also C49.1, U19.1 (OUT)
- net +5V: now also C34.1, C48.1, C51.1, U19.3 (EN), U19.4 (IN), U20.A2 (IN)
- net GND: now also C34.2, C48.2, C49.2, C51.2, C59.2, C60.2, C61.2, C62.2, C63.2, U19.2 (GND), U19.5 (GND), U20.B1 (GND), U21.B1 (GND), U22.B1 (GND)
- net TRANS_FB: now also U10.1 (FB)
- net TRANS_VCC: now also C60.1, C62.1, U21.A2 (IN), U22.A2 (IN)
- net TRANS_VREF: no longer U10.1 (FB)
- new net +5V_OUT: C59.1, U20.A1 (OUT)
- new net PORT_EN: U22.B2 (ON)
- new net P_EN: U20.B2 (ON), U21.B2 (ON)
- new net TRANS_VCC_OUT: C61.1, U21.A1 (OUT)
- new net VEE: C63.1, U22.A1 (OUT)
