File: projects/HSLink-Pro/hardware/Interface.kicad_sch (KiCad schematic)
At the start: 19 parts, among them J1 IDC 2x10p 夹板, J2 USB_C_Receptacle_USB2.0, Q1 AO3401A, Q2 2N7002, Q3 AO3401A, Q4 2N7002, U14 MT9700, U15 ESD0524P, U16 ESD0524P, U17 ESD0524P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

Commit message: update: 更新原理图
Parts:
- removed Q1, Q3: AO3401A, Package_TO_SOT_SMD:SOT-23, symbol Transistor_FET:AO3401A
- removed Q2, Q4: 2N7002, Package_TO_SOT_SMD:SOT-323_SC-70, symbol Transistor_FET:2N7002
- removed R19, R20: 100k, Resistor_SMD:R_0402_1005Metric, symbol Device:R
